Commit message: Modified robot_base.xacro

File: src/description/urdf/robot_base.xacro (robot description, xacro)
@@ -40,4 +40,29 @@
     <self_collide>false</self_collide>
   </gazebo>
+  <!-- ================= IMU LINK ================= -->
+<link name="imu_link"/>
+<joint name="imu_joint" type="fixed">
+  <parent link="base_link"/>
+  <child link="imu_link"/>
+  <origin xyz="0 0 0.15"/>
+</joint>
+<gazebo reference="imu_link">
+  <sensor name="imu_sensor_2" type="imu">
+    <always_on>true</always_on>
+    <update_rate>100</update_rate>
+    <imu>
+      <angular_velocity>
+        <x>true</x>
+        <y>true</y>
+        <z>true</z>
+      </angular_velocity>
+      <linear_acceleration>
+        <x>true</x>
+        <y>true</y>
+        <z>true</z>
+      </linear_acceleration>
+    </imu>
+  </sensor>
+</gazebo>
   <!-- ================= WHEEL MACRO ================= -->
   <xacro:macro name="wheel" params="name x y">

Commit message: odom and imu working perfectly, tested

File: src/description/urdf/robot_base.xacro (robot description, xacro)
@@ -40,6 +40,8 @@
     <self_collide>false</self_collide>
   </gazebo>
-  <!-- ================= IMU LINK ================= -->
-<link name="imu_link"/>
+<!-- ================= IMU LINK ================= -->
+<link name="imu_link">
+  <origin xyz="0 0 0.15" rpy="0 0 0"/>
+</link>
 <joint name="imu_joint" type="fixed">
   <parent link="base_link"/>
@@ -47,22 +49,4 @@
   <origin xyz="0 0 0.15"/>
 </joint>
-<gazebo reference="imu_link">
-  <sensor name="imu_sensor_2" type="imu">
-    <always_on>true</always_on>
-    <update_rate>100</update_rate>
-    <imu>
-      <angular_velocity>
-        <x>true</x>
-        <y>true</y>
-        <z>true</z>
-      </angular_velocity>
-      <linear_acceleration>
-        <x>true</x>
-        <y>true</y>
-        <z>true</z>
-      </linear_acceleration>
-    </imu>
-  </sensor>
-</gazebo>
   <!-- ================= WHEEL MACRO ================= -->
   <xacro:macro name="wheel" params="name x y">

File: src/description/urdf/robot_sensors.xacro (robot description, xacro)
@@ -2,39 +2,65 @@
 <robot xmlns:xacro="http://www.ros.org/wiki/xacro">
   <xacro:macro name="sensors">
-    <!-- ================= IMU ================= -->
-    <gazebo reference="base_link">
-      <sensor name="imu_sensor" type="imu">
-        <always_on>true</always_on>
-        <update_rate>100</update_rate>
-        <topic>/imu</topic>
-        <imu>
-          <angular_velocity>
-            <x>true</x>
-            <y>true</y>
-            <z>true</z>
-          </angular_velocity>
-          <linear_acceleration>
-            <x>true</x>
-            <y>true</y>
-            <z>true</z>
-          </linear_acceleration>
-        </imu>
-        <plugin
-          filename="gz-sim-imu-system"
-          name="gz::sim::systems::Imu"/>
-      </sensor>
-    </gazebo>
-    <!-- ================= GPS ================= -->
-    <gazebo reference="base_link">
-      <sensor name="gps_sensor" type="navsat">
-        <always_on>true</always_on>
-        <update_rate>10</update_rate>
-        <topic>/gps</topic>
-        <plugin
-          filename="gz-sim-navsat-system"
-          name="gz::sim::systems::NavSat"/>
-      </sensor>
-    </gazebo>
-    <!-- ================= LIDAR ================= -->
+ <!-- ================= IMU ================= -->
+<!-- Fixed IMU with proper noise and frame configuration -->
+<gazebo reference="imu_link">
+  <sensor name="imu_sensor" type="imu">
+    <always_on>true</always_on>
+    <update_rate>100</update_rate>
+    <topic>/imu</topic>
+    <!-- Orientation -->
+    <orientation>true</orientation>
+    <imu>
+      <angular_velocity>
+        <x>true</x>
+        <y>true</y>
+        <z>true</z>
+      </angular_velocity>
+      <linear_acceleration>
+        <x>true</x>
+        <y>true</y>
+        <z>true</z>
+      </linear_acceleration>
+    </imu>
+    <!-- Plugin for IMU simulation -->
+    <plugin
+      filename="gz-sim-imu-system"
+      name="gz::sim::systems::Imu">
+      <ros_namespace>/imu</ros_namespace>
+      <frame_id>imu_link</frame_id>
+    </plugin>
+  </sensor>
+</gazebo>
+<!-- ================= GPS ================= -->
+<gazebo reference="base_link">
+  <sensor name="gps_sensor" type="navsat">
+    <always_on>true</always_on>
+    <update_rate>10</update_rate>
+    <topic>/gps</topic>
+    <!-- Position-only sensor (not velocity) -->
+    <position>true</position>
+    <velocity>false</velocity>
+    <!-- Add some noise for realism -->
+    <noise type="gaussian">
+      <rate>0.0 0.0 0.0</rate>
+      <position>0.0 0.0 0.0</position>
+    </noise>
+    <navsat>
+      <position_sensing>true</position_sensing>
+      <velocity_sensing>false</velocity_sensing>
+    </navsat>
+    <plugin
+      filename="gz-sim-navsat-system"
+      name="gz::sim::systems::NavSat">
+      <ros_namespace>/gps</ros_namespace>
+      <frame_id>gps_link</frame_id>
+      <latitude_deg>0.0</latitude_deg>
+      <longitude_deg>0.0</longitude_deg>
+      <altitude>0.0</altitude>
+      <heading_offset>0.0</heading_offset>
+    </plugin>
+  </sensor>
+</gazebo>
+<!-- ================= LIDAR ================= -->
 <gazebo reference="base_link">
   <sensor name="lidar_sensor" type="gpu_lidar">
@@ -42,5 +68,4 @@
     <update_rate>10</update_rate>
     <topic>/scan</topic>
-    <gz_frame_id>base_link</gz_frame_id>
     <lidar>
       <scan>
@@ -57,9 +82,16 @@
         <resolution>0.01</resolution>
       </range>
+      <noise>
+        <type>gaussian</type>
+        <mean>0.0</mean>
+        <stddev>0.01</stddev>
+      </noise>
     </lidar>
     <plugin
-      filename="gz-sim-sensors-system"
-      name="gz::sim::systems::Sensors">
-      <render_engine>ogre2</render_engine>
+      filename="gz-sim-lidar-system"
+      name="gz::sim::systems::Lidar">
+      <ros_namespace>/scan</ros_namespace>
+      <frame_id>lidar_link</frame_id>
+      <topic>/scan</topic>
     </plugin>
   </sensor>

Commit message: gps, odom and imu working perfectly, tested

File: src/description/urdf/robot_base.xacro (robot description, xacro)
@@ -10,4 +10,11 @@
   <xacro:property name="wheel_x_offset" value="0.18"/>
   <xacro:property name="wheel_y_offset" value="0.22"/>
+    <!-- ================= BASE FOOTPRINT ================= -->
+<link name="base_footprint"/>
+<joint name="base_footprint_joint" type="fixed">
+  <parent link="base_footprint"/>
+  <child link="base_link"/>
+  <origin xyz="0 0 0" rpy="0 0 0"/>
+</joint>
   <!-- ================= BASE LINK ================= -->
   <link name="base_link">
@@ -40,13 +47,31 @@
     <self_collide>false</self_collide>
   </gazebo>
-<!-- ================= IMU LINK ================= -->
-<link name="imu_link">
-  <origin xyz="0 0 0.15" rpy="0 0 0"/>
-</link>
-<joint name="imu_joint" type="fixed">
-  <parent link="base_link"/>
-  <child link="imu_link"/>
-  <origin xyz="0 0 0.15"/>
-</joint>
+  <!-- ================= IMU LINK ================= -->
+  <link name="imu_link">
+    <origin xyz="0 0 0.15" rpy="0 0 0"/>
+  </link>
+  <joint name="imu_joint" type="fixed">
+    <parent link="base_link"/>
+    <child link="imu_link"/>
+    <origin xyz="0 0 0.15"/>
+  </joint>
+  <!-- ================= GPS LINK ================= -->
+  <link name="gps_link">
+    <origin xyz="0 0 0.1" rpy="0 0 0"/>
+  </link>
+  <joint name="gps_joint" type="fixed">
+    <parent link="base_link"/>
+    <child link="gps_link"/>
+    <origin xyz="0 0 0.1"/>
+  </joint>
+  <!-- ================= LIDAR LINK ================= -->
+  <link name="lidar_link">
+    <origin xyz="0.2 0 0.15" rpy="0 0 0"/>
+  </link>
+  <joint name="lidar_joint" type="fixed">
+    <parent link="base_link"/>
+    <child link="lidar_link"/>
+    <origin xyz="0.2 0 0.15"/>
+  </joint>
   <!-- ================= WHEEL MACRO ================= -->
   <xacro:macro name="wheel" params="name x y">

File: src/description/urdf/robot_sensors.xacro (robot description, xacro)
@@ -2,99 +2,44 @@
 <robot xmlns:xacro="http://www.ros.org/wiki/xacro">
   <xacro:macro name="sensors">
- <!-- ================= IMU ================= -->
-<!-- Fixed IMU with proper noise and frame configuration -->
-<gazebo reference="imu_link">
-  <sensor name="imu_sensor" type="imu">
-    <always_on>true</always_on>
-    <update_rate>100</update_rate>
-    <topic>/imu</topic>
-    <!-- Orientation -->
-    <orientation>true</orientation>
-    <imu>
-      <angular_velocity>
-        <x>true</x>
-        <y>true</y>
-        <z>true</z>
-      </angular_velocity>
-      <linear_acceleration>
-        <x>true</x>
-        <y>true</y>
-        <z>true</z>
-      </linear_acceleration>
-    </imu>
-    <!-- Plugin for IMU simulation -->
-    <plugin
-      filename="gz-sim-imu-system"
-      name="gz::sim::systems::Imu">
-      <ros_namespace>/imu</ros_namespace>
-      <frame_id>imu_link</frame_id>
-    </plugin>
-  </sensor>
-</gazebo>
-<!-- ================= GPS ================= -->
-<gazebo reference="base_link">
-  <sensor name="gps_sensor" type="navsat">
-    <always_on>true</always_on>
-    <update_rate>10</update_rate>
-    <topic>/gps</topic>
-    <!-- Position-only sensor (not velocity) -->
-    <position>true</position>
-    <velocity>false</velocity>
-    <!-- Add some noise for realism -->
-    <noise type="gaussian">
-      <rate>0.0 0.0 0.0</rate>
-      <position>0.0 0.0 0.0</position>
-    </noise>
-    <navsat>
-      <position_sensing>true</position_sensing>
-      <velocity_sensing>false</velocity_sensing>
-    </navsat>
-    <plugin
-      filename="gz-sim-navsat-system"
-      name="gz::sim::systems::NavSat">
-      <ros_namespace>/gps</ros_namespace>
-      <frame_id>gps_link</frame_id>
-      <latitude_deg>0.0</latitude_deg>
-      <longitude_deg>0.0</longitude_deg>
-      <altitude>0.0</altitude>
-      <heading_offset>0.0</heading_offset>
-    </plugin>
-  </sensor>
-</gazebo>
-<!-- ================= LIDAR ================= -->
-<gazebo reference="base_link">
-  <sensor name="lidar_sensor" type="gpu_lidar">
-    <always_on>true</always_on>
-    <update_rate>10</update_rate>
-    <topic>/scan</topic>
-    <lidar>
-      <scan>
-        <horizontal>
-          <samples>720</samples>
-          <resolution>1</resolution>
-          <min_angle>-3.14159</min_angle>
-          <max_angle>3.14159</max_angle>
-        </horizontal>
-      </scan>
-      <range>
-        <min>0.1</min>
-        <max>10.0</max>
-        <resolution>0.01</resolution>
-      </range>
-      <noise>
-        <type>gaussian</type>
-        <mean>0.0</mean>
-        <stddev>0.01</stddev>
-      </noise>
-    </lidar>
-    <plugin
-      filename="gz-sim-lidar-system"
-      name="gz::sim::systems::Lidar">
-      <ros_namespace>/scan</ros_namespace>
-      <frame_id>lidar_link</frame_id>
-      <topic>/scan</topic>
-    </plugin>
-  </sensor>
-</gazebo>
+    <!-- ================= IMU ================= -->
+    <gazebo reference="imu_link">
+      <sensor name="imu_sensor" type="imu">
+        <always_on>true</always_on>
+        <update_rate>100</update_rate>
+        <topic>/imu</topic>
+        <gz_frame_id>imu_link</gz_frame_id>
+      </sensor>
+    </gazebo>
+    <!-- ================= GPS (FIXED PROPERLY) ================= -->
+    <gazebo reference="gps_link">
+      <sensor name="gps_sensor" type="navsat">
+        <always_on>true</always_on>
+        <update_rate>5</update_rate>
+        <topic>/gps</topic>
+        <gz_frame_id>gps_link</gz_frame_id>
+      </sensor>
+    </gazebo>
+    <!-- ================= LIDAR (CPU SAFE VERSION) ================= -->
+    <gazebo reference="lidar_link">
+      <sensor name="lidar_sensor" type="lidar">
+        <always_on>true</always_on>
+        <update_rate>10</update_rate>
+        <topic>/scan</topic>
+        <gz_frame_id>lidar_link</gz_frame_id>
+        <lidar>
+          <scan>
+            <horizontal>
+              <samples>720</samples>
+              <min_angle>-3.14159</min_angle>
+              <max_angle>3.14159</max_angle>
+            </horizontal>
+          </scan>
+          <range>
+            <min>0.1</min>
+            <max>10.0</max>
+          </range>
+        </lidar>
+      </sensor>
+    </gazebo>
   </xacro:macro>
 </robot>

File: src/description/urdf/robot_sim.xacro (robot description, xacro)
@@ -2,12 +2,9 @@
 <robot xmlns:xacro="http://www.ros.org/wiki/xacro">
   <xacro:macro name="sim">
-    <!-- ================= DIFF DRIVE PLUGIN ================= -->
     <gazebo>
   <plugin filename="gz-sim-diff-drive-system"
           name="gz::sim::systems::DiffDrive">
-    <!-- Left wheels -->
     <left_joint>front_left_wheel_joint</left_joint>
     <left_joint>rear_left_wheel_joint</left_joint>
-    <!-- Right wheels -->
     <right_joint>front_right_wheel_joint</right_joint>
     <right_joint>rear_right_wheel_joint</right_joint>
@@ -17,5 +14,5 @@
     <odom_topic>/odom</odom_topic>
     <frame_id>odom</frame_id>
-    <child_frame_id>base_link</child_frame_id>
+    <child_frame_id>base_footprint</child_frame_id>
   </plugin>
 </gazebo>

Commit message: RGB camera, LiDar,gps, odom and imu working perfectly, tested

File: src/description/urdf/robot_base.xacro (robot description, xacro)
@@ -74,4 +74,13 @@
     <origin xyz="0.2 0 0.15"/>
   </joint>
+  <!-- ================= CAMERA LINK ================= -->
+  <link name="camera_link">
+    <origin xyz="0.15 0 0.12" rpy="0 0 0"/>
+  </link>
+  <joint name="camera_joint" type="fixed">
+    <parent link="base_link"/>
+    <child link="camera_link"/>
+    <origin xyz="0.15 0 0.12"/>
+  </joint>
   <!-- ================= WHEEL MACRO ================= -->
   <xacro:macro name="wheel" params="name x y">

File: src/description/urdf/robot_sensors.xacro (robot description, xacro)
@@ -18,5 +18,5 @@
       </sensor>
     </gazebo>
-    <!-- ================= LIDAR (FIXED) ================= -->
+    <!-- ================= LIDAR ================= -->
     <gazebo reference="lidar_link">
       <sensor name="lidar_sensor" type="gpu_lidar">
@@ -39,10 +39,25 @@
             <resolution>0.01</resolution>
           </range>
-          <noise>
-            <type>gaussian</type>
-            <mean>0.0</mean>
-            <stddev>0.01</stddev>
-          </noise>
         </lidar>
+      </sensor>
+    </gazebo>
+    <!-- ================= CAMERA ================= -->
+    <gazebo reference="camera_link">
+      <sensor name="camera_sensor" type="camera">
+        <always_on>true</always_on>
+        <update_rate>30</update_rate>
+        <topic>/camera/image_raw</topic>
+        <camera>
+          <horizontal_fov>1.047</horizontal_fov>
+          <image>
+            <width>640</width>
+            <height>480</height>
+            <format>R8G8B8</format>
+          </image>
+          <clip>
+            <near>0.1</near>
+            <far>100</far>
+          </clip>
+        </camera>
       </sensor>
     </gazebo>
